File: kicad/brakeUnwindControl.sch (KiCad schematic (older format))
At the start: 12 parts

Commit message: KICAD: Modificar brakeUnwindControl.sch
Parts:
- D20: renamed from D?; value (none) -> ~
- J73, J74: renamed from J?; value (none) -> ~
- Q16: value (none) -> ~
- Q17: renamed from Q?; value (none) -> ~
- R39, R40, R41, R42, R43, R44: renamed from R?; value (none) -> ~
- U15: renamed from U?; value (none) -> ~
Changed lines of the file:
@@
 AR Path="/5F888A13/601F3393" Ref="Q?"  Part="1"
 AR Path="/5FBD1D9A/601F3393" Ref="Q?"  Part="1"
+AR Path="/5FBD1D9A/601CE166/601F3393" Ref="Q17"  Part="1"
 F 0 "Q17" H 7054 3896 50  0000 L CNN
-F 1 "" H 6850 3850 50  0001 C CNN
+F 1 "~" H 6850 3850 50  0001 C CNN
 F 2 "Package_TO_SOT_THT:TO-220-3_Vertical" H 7100 3775 50  0001 L CIN
 F 3 "http://www.irf.com/product-info/datasheets/data/irlz44n.pdf" H 6850 3850 50  0001 L CNN
@@
 AR Path="/5F888A13/601F3399" Ref="U?"  Part="1"
 AR Path="/5FBD1D9A/601F3399" Ref="U?"  Part="1"
+AR Path="/5FBD1D9A/601CE166/601F3399" Ref="U15"  Part="1"
 F 0 "U15" H 5550 4075 50  0000 C CNN
-F 1 "" H 5550 3750 50  0001 C CNN
+F 1 "~" H 5550 3750 50  0001 C CNN
 F 2 "Package_DIP:DIP-6_W7.62mm" H 5350 3550 50  0001 L CIN
 F 3 "https://www.vishay.com/docs/81181/4n35.pdf" H 5550 3750 50  0001 L CNN
@@
 AR Path="/5F888A13/601F339F" Ref="R?"  Part="1"
 AR Path="/5FBD1D9A/601F339F" Ref="R?"  Part="1"
+AR Path="/5FBD1D9A/601CE166/601F339F" Ref="R43"  Part="1"
 F 0 "R43" V 6550 4150 50  0000 C CNN
-F 1 "" H 6650 4150 50  0001 C CNN
+F 1 "~" H 6650 4150 50  0001 C CNN
 F 2 "Resistor_THT:R_Axial_DIN0207_L6.3mm_D2.5mm_P7.62mm_Horizontal" V 6580 4150 50  0001 C CNN
 F 3 "~" H 6650 4150 50  0001 C CNN
@@
 AR Path="/5F888A13/601F33A6" Ref="R?"  Part="1"
 AR Path="/5FBD1D9A/601F33A6" Ref="R?"  Part="1"
+AR Path="/5FBD1D9A/601CE166/601F33A6" Ref="R42"  Part="1"
 F 0 "R42" V 6350 3850 50  0000 C CNN
-F 1 "" H 6250 3850 50  0001 C CNN
+F 1 "~" H 6250 3850 50  0001 C CNN
 F 2 "Resistor_THT:R_Axial_DIN0207_L6.3mm_D2.5mm_P7.62mm_Horizontal" V 6180 3850 50  0001 C CNN
 F 3 "~" H 6250 3850 50  0001 C CNN
@@
 AR Path="/5F888A13/601F33AF" Ref="D?"  Part="1"
 AR Path="/5FBD1D9A/601F33AF" Ref="D?"  Part="1"
+AR Path="/5FBD1D9A/601CE166/601F33AF" Ref="D20"  Part="1"
 F 0 "D20" H 5843 4667 50  0000 C CNN
-F 1 "" H 5850 4450 50  0001 C CNN
+F 1 "~" H 5850 4450 50  0001 C CNN
 F 2 "LED_THT:LED_D5.0mm" H 5850 4450 50  0001 C CNN
 F 3 "~" H 5850 4450 50  0001 C CNN
@@
 AR Path="/5F888A13/601F33B5" Ref="R?"  Part="1"
 AR Path="/5FBD1D9A/601F33B5" Ref="R?"  Part="1"
+AR Path="/5FBD1D9A/601CE166/601F33B5" Ref="R40"  Part="1"
 F 0 "R40" V 5150 3300 50  0000 C CNN
-F 1 "" H 5250 3300 50  0001 C CNN
+F 1 "~" H 5250 3300 50  0001 C CNN
 F 2 "Resistor_THT:R_Axial_DIN0207_L6.3mm_D2.5mm_P7.62mm_Horizontal" V 5180 3300 50  0001 C CNN
 F 3 "~" H 5250 3300 50  0001 C CNN
@@
 AR Path="/5F888A13/601F33BF" Ref="R?"  Part="1"
 AR Path="/5FBD1D9A/601F33BF" Ref="R?"  Part="1"
+AR Path="/5FBD1D9A/601CE166/601F33BF" Ref="R41"  Part="1"
 F 0 "R41" V 5750 4150 50  0000 C CNN
-F 1 "" H 5850 4150 50  0001 C CNN
+F 1 "~" H 5850 4150 50  0001 C CNN
 F 2 "Resistor_THT:R_Axial_DIN0207_L6.3mm_D2.5mm_P7.62mm_Horizontal" V 5780 4150 50  0001 C CNN
 F 3 "~" H 5850 4150 50  0001 C CNN
@@
 AR Path="/5F888A13/601F33C6" Ref="J?"  Part="1"
 AR Path="/5FBD1D9A/601F33C6" Ref="J?"  Part="1"
+AR Path="/5FBD1D9A/601CE166/601F33C6" Ref="J74"  Part="1"
 F 0 "J74" H 8000 3300 50  0000 C CNN
-F 1 "" H 8000 3600 50  0001 C CNN
+F 1 "~" H 8000 3600 50  0001 C CNN
 F 2 "TerminalBlock_Altech:Altech_AK300_1x03_P5.00mm_45-Degree" H 8000 3600 50  0001 C CNN
 F 3 "~" H 8000 3600 50  0001 C CNN
@@
 AR Path="/5F888A13/601F33CD" Ref="R?"  Part="1"
 AR Path="/5FBD1D9A/601F33CD" Ref="R?"  Part="1"
+AR Path="/5FBD1D9A/601CE166/601F33CD" Ref="R39"  Part="1"
 F 0 "R39" H 4550 4100 50  0000 C CNN
-F 1 "" H 4650 4100 50  0001 C CNN
+F 1 "~" H 4650 4100 50  0001 C CNN
 F 2 "Resistor_THT:R_Axial_DIN0207_L6.3mm_D2.5mm_P7.62mm_Horizontal" V 4580 4100 50  0001 C CNN
 F 3 "~" H 4650 4100 50  0001 C CNN
@@
 AR Path="/5F888A13/601F33DC" Ref="R?"  Part="1"
 AR Path="/5FBD1D9A/601F33DC" Ref="R?"  Part="1"
+AR Path="/5FBD1D9A/601CE166/601F33DC" Ref="R44"  Part="1"
 F 0 "R44" V 7050 3200 50  0000 C CNN
-F 1 "" H 6950 3200 50  0001 C CNN
+F 1 "~" H 6950 3200 50  0001 C CNN
 F 2 "Resistor_THT:R_Axial_DIN0207_L6.3mm_D2.5mm_P7.62mm_Horizontal" V 6880 3200 50  0001 C CNN
 F 3 "~" H 6950 3200 50  0001 C CNN
@@
 P 5150 4250
 F 0 "Q16" H 5340 4204 50  0000 L CNN
-F 1 "" H 5150 4250 50  0001 C CNN
+F 1 "~" H 5150 4250 50  0001 C CNN
 F 2 "Package_TO_SOT_THT:TO-92_Inline" H 5350 4175 50  0001 L CIN
 F 3 "https://www.fairchildsemi.com/datasheets/2N/2N3906.pdf" H 5150 4250 50  0001 L CNN
@@
 AR Path="/5F888A13/601F33F0" Ref="J?"  Part="1"
 AR Path="/5FBD1D9A/601F33F0" Ref="J?"  Part="1"
+AR Path="/5FBD1D9A/601CE166/601F33F0" Ref="J73"  Part="1"
 F 0 "J73" H 3600 4150 50  0000 C CNN
-F 1 "" H 3600 3850 50  0001 C CNN
+F 1 "~" H 3600 3850 50  0001 C CNN
 F 2 "TerminalBlock_Altech:Altech_AK300_1x03_P5.00mm_45-Degree" H 3600 3850 50  0001 C CNN
 F 3 "~" H 3600 3850 50  0001 C CNN
