File: kicad/brakeUnwindControl.sch (KiCad schematic (older format))
At the start: 12 parts

Commit message: KICAD: Guardar cambios sch de los controles de los cluches y freno
Other:
- note added: "Azul"
- note added: "Blanco/Azul"
- note added: "brakeUnwindControl"
Changed lines of the file:
@@
 Sheet 19 22
 Title "Mainet-mega -- brakeUnwindControl"
-Date "2021-04-07"
+Date "2021-07-09"
 Rev "1.0"
 Comp "Tovenca"
@@
 Text Label 7600 4750 0    50   ~ 0
 0V
+Text Notes 7050 3600 0    50   ~ 0
+brakeUnwindControl
+Text Notes 8200 3500 0    50   ~ 0
+Azul
+Text Notes 8200 3700 0    50   ~ 0
+Blanco/Azul
 $EndSCHEMATC

Commit message: KICAD: Agregar cvambios .sch controles tarjetas MP
Other:
- note added: "D12 (brakeUnwindControl)"
- note added: "GNDD"
- note added: "VCC"
Changed lines of the file:
@@
 Sheet 19 22
 Title "Mainet-mega -- brakeUnwindControl"
-Date "2021-07-09"
+Date "2021-07-13"
 Rev "1.0"
 Comp "Tovenca"
@@
 Text Notes 8200 3700 0    50   ~ 0
 Blanco/Azul
+Text Notes 2500 3900 0    50   ~ 0
+D12 (brakeUnwindControl)
+Text Notes 2500 4000 0    50   ~ 0
+GNDD
+Text Notes 2500 3800 0    50   ~ 0
+VCC
 $EndSCHEMATC
