File: kicad/lowerClutchControl.sch (KiCad schematic (older format))
At the start: 12 parts

Commit message: KICAD: Modificar lowerClutchControl.sch
Parts:
- D18: renamed from D?; value (none) -> ~
- J69, J70: renamed from J?; value (none) -> ~
- Q12: value (none) -> ~
- Q13: renamed from Q?; value (none) -> ~
- R27, R28, R29, R30, R31, R32: renamed from R?; value (none) -> ~
- U13: renamed from U?; value (none) -> ~
Changed lines of the file:
@@
 AR Path="/5F888A13/601F1261" Ref="Q?"  Part="1"
 AR Path="/5FBD1D9A/601F1261" Ref="Q?"  Part="1"
+AR Path="/5FBD1D9A/601BF406/601F1261" Ref="Q13"  Part="1"
 F 0 "Q13" H 7254 3446 50  0000 L CNN
-F 1 "" H 7050 3400 50  0001 C CNN
+F 1 "~" H 7050 3400 50  0001 C CNN
 F 2 "Package_TO_SOT_THT:TO-220-3_Vertical" H 7300 3325 50  0001 L CIN
 F 3 "http://www.irf.com/product-info/datasheets/data/irlz44n.pdf" H 7050 3400 50  0001 L CNN
@@
 AR Path="/5F888A13/601F1267" Ref="U?"  Part="1"
 AR Path="/5FBD1D9A/601F1267" Ref="U?"  Part="1"
+AR Path="/5FBD1D9A/601BF406/601F1267" Ref="U13"  Part="1"
 F 0 "U13" H 5750 3625 50  0000 C CNN
-F 1 "" H 5750 3300 50  0001 C CNN
+F 1 "~" H 5750 3300 50  0001 C CNN
 F 2 "Package_DIP:DIP-6_W7.62mm" H 5550 3100 50  0001 L CIN
 F 3 "https://www.vishay.com/docs/81181/4n35.pdf" H 5750 3300 50  0001 L CNN
@@
 AR Path="/5F888A13/601F126D" Ref="R?"  Part="1"
 AR Path="/5FBD1D9A/601F126D" Ref="R?"  Part="1"
+AR Path="/5FBD1D9A/601BF406/601F126D" Ref="R31"  Part="1"
 F 0 "R31" V 6750 3700 50  0000 C CNN
-F 1 "" H 6850 3700 50  0001 C CNN
+F 1 "~" H 6850 3700 50  0001 C CNN
 F 2 "Resistor_THT:R_Axial_DIN0207_L6.3mm_D2.5mm_P7.62mm_Horizontal" V 6780 3700 50  0001 C CNN
 F 3 "~" H 6850 3700 50  0001 C CNN
@@
 AR Path="/5F888A13/601F1274" Ref="R?"  Part="1"
 AR Path="/5FBD1D9A/601F1274" Ref="R?"  Part="1"
+AR Path="/5FBD1D9A/601BF406/601F1274" Ref="R30"  Part="1"
 F 0 "R30" V 6550 3400 50  0000 C CNN
-F 1 "" H 6450 3400 50  0001 C CNN
+F 1 "~" H 6450 3400 50  0001 C CNN
 F 2 "Resistor_THT:R_Axial_DIN0207_L6.3mm_D2.5mm_P7.62mm_Horizontal" V 6380 3400 50  0001 C CNN
 F 3 "~" H 6450 3400 50  0001 C CNN
@@
 AR Path="/5F888A13/601F127D" Ref="D?"  Part="1"
 AR Path="/5FBD1D9A/601F127D" Ref="D?"  Part="1"
+AR Path="/5FBD1D9A/601BF406/601F127D" Ref="D18"  Part="1"
 F 0 "D18" H 6043 4217 50  0000 C CNN
-F 1 "" H 6050 4000 50  0001 C CNN
+F 1 "~" H 6050 4000 50  0001 C CNN
 F 2 "LED_THT:LED_D5.0mm" H 6050 4000 50  0001 C CNN
 F 3 "~" H 6050 4000 50  0001 C CNN
@@
 AR Path="/5F888A13/601F1283" Ref="R?"  Part="1"
 AR Path="/5FBD1D9A/601F1283" Ref="R?"  Part="1"
+AR Path="/5FBD1D9A/601BF406/601F1283" Ref="R28"  Part="1"
 F 0 "R28" V 5350 2850 50  0000 C CNN
-F 1 "" H 5450 2850 50  0001 C CNN
+F 1 "~" H 5450 2850 50  0001 C CNN
 F 2 "Resistor_THT:R_Axial_DIN0207_L6.3mm_D2.5mm_P7.62mm_Horizontal" V 5380 2850 50  0001 C CNN
 F 3 "~" H 5450 2850 50  0001 C CNN
@@
 AR Path="/5F888A13/601F128D" Ref="R?"  Part="1"
 AR Path="/5FBD1D9A/601F128D" Ref="R?"  Part="1"
+AR Path="/5FBD1D9A/601BF406/601F128D" Ref="R29"  Part="1"
 F 0 "R29" V 5950 3700 50  0000 C CNN
-F 1 "" H 6050 3700 50  0001 C CNN
+F 1 "~" H 6050 3700 50  0001 C CNN
 F 2 "Resistor_THT:R_Axial_DIN0207_L6.3mm_D2.5mm_P7.62mm_Horizontal" V 5980 3700 50  0001 C CNN
 F 3 "~" H 6050 3700 50  0001 C CNN
@@
 AR Path="/5F888A13/601F1294" Ref="J?"  Part="1"
 AR Path="/5FBD1D9A/601F1294" Ref="J?"  Part="1"
+AR Path="/5FBD1D9A/601BF406/601F1294" Ref="J70"  Part="1"
 F 0 "J70" H 8200 2850 50  0000 C CNN
-F 1 "" H 8200 3150 50  0001 C CNN
+F 1 "~" H 8200 3150 50  0001 C CNN
 F 2 "TerminalBlock_Altech:Altech_AK300_1x03_P5.00mm_45-Degree" H 8200 3150 50  0001 C CNN
 F 3 "~" H 8200 3150 50  0001 C CNN
@@
 AR Path="/5F888A13/601F129B" Ref="R?"  Part="1"
 AR Path="/5FBD1D9A/601F129B" Ref="R?"  Part="1"
+AR Path="/5FBD1D9A/601BF406/601F129B" Ref="R27"  Part="1"
 F 0 "R27" H 4750 3650 50  0000 C CNN
-F 1 "" H 4850 3650 50  0001 C CNN
+F 1 "~" H 4850 3650 50  0001 C CNN
 F 2 "Resistor_THT:R_Axial_DIN0207_L6.3mm_D2.5mm_P7.62mm_Horizontal" V 4780 3650 50  0001 C CNN
 F 3 "~" H 4850 3650 50  0001 C CNN
@@
 AR Path="/5F888A13/601F12AA" Ref="R?"  Part="1"
 AR Path="/5FBD1D9A/601F12AA" Ref="R?"  Part="1"
+AR Path="/5FBD1D9A/601BF406/601F12AA" Ref="R32"  Part="1"
 F 0 "R32" V 7250 2750 50  0000 C CNN
-F 1 "" H 7150 2750 50  0001 C CNN
+F 1 "~" H 7150 2750 50  0001 C CNN
 F 2 "Resistor_THT:R_Axial_DIN0207_L6.3mm_D2.5mm_P7.62mm_Horizontal" V 7080 2750 50  0001 C CNN
 F 3 "~" H 7150 2750 50  0001 C CNN
@@
 P 5350 3800
 F 0 "Q12" H 5540 3754 50  0000 L CNN
-F 1 "" H 5350 3800 50  0001 C CNN
+F 1 "~" H 5350 3800 50  0001 C CNN
 F 2 "Package_TO_SOT_THT:TO-92_Inline" H 5550 3725 50  0001 L CIN
 F 3 "https://www.fairchildsemi.com/datasheets/2N/2N3906.pdf" H 5350 3800 50  0001 L CNN
@@
 AR Path="/5F888A13/601F12BE" Ref="J?"  Part="1"
 AR Path="/5FBD1D9A/601F12BE" Ref="J?"  Part="1"
+AR Path="/5FBD1D9A/601BF406/601F12BE" Ref="J69"  Part="1"
 F 0 "J69" H 3800 3700 50  0000 C CNN
-F 1 "" H 3800 3400 50  0001 C CNN
+F 1 "~" H 3800 3400 50  0001 C CNN
 F 2 "TerminalBlock_Altech:Altech_AK300_1x03_P5.00mm_45-Degree" H 3800 3400 50  0001 C CNN
 F 3 "~" H 3800 3400 50  0001 C CNN
