File: kicad/mainet-mega-relay-driver-8.sch (KiCad schematic (older format))
At the start: 8 parts, among them J37 Screw_Terminal_01x03, K8 SANYOU_SRD_Form_C, Q8 2N3904, U9 4N37

Commit message: KICAD: Actualizar archivos del módulo de relés
Other:
- note added: "Relay Ground\nNo conectar a la tierra\ndel Arduino Mega\n"
- note removed: "No conectar a la tierra del Arduino Mega\n"
- note removed: "Relay Ground\n"
Changed lines of the file:
@@
 EESchema Schematic File Version 4
+LIBS:mainet-mega-cache
 EELAYER 30 0
 EELAYER END
 $Descr A4 11693 8268
 encoding utf-8
-Sheet 14 21
+Sheet 14 22
 Title "Mainet-mega -- "
 Date "2021-04-07"
@@
 	1    0    0    -1
 $EndComp
-Text Notes 6500 4600 0    50   ~ 0
-Relay Ground\n
-Text Notes 6500 4700 0    50   ~ 0
-No conectar a la tierra del Arduino Mega\n
 NoConn ~ 5400 4100
 Wire Wire Line
@@
 Text Notes 3150 2600 0    50   ~ 0
 VCC:\nSalida +5V del Arduino
+Text Notes 3600 3900 0    50   ~ 0
+Relay Ground\nNo conectar a la tierra\ndel Arduino Mega\n
+Text Notes 6000 5000 0    50   ~ 0
+Relay Ground\nNo conectar a la tierra\ndel Arduino Mega\n
 $EndSCHEMATC
