File: kicad/mainet-mega-relay-driver-3.sch (KiCad schematic (older format))
At the start: 8 parts, among them J36 Screw_Terminal_01x03, K3 SANYOU_SRD_Form_C, Q3 2N3904, U4 4N37

Commit message: KICAD: Modificar esquemático
Parts:
- added J86, J87: Conn_01x01_Male, symbol Connector:Conn_01x01_Male
Connections:
- net labels added: +24V, C3, Digital_input_4, NC3, NO3
- net labels removed: C1, NC1, NO1
- wire segments 28 -> 31
Other:
- note added: "3er relé de izquierda a derecha"
- note added: "D19-runReverseControl"
- note added: "Terminal 13 del M400"
Changed lines of the file:
@@
 EESchema Schematic File Version 4
+LIBS:mainet-mega-cache
 EELAYER 30 0
 EELAYER END
 $Descr A4 11693 8268
 encoding utf-8
-Sheet 1 1
-Title ""
-Date ""
-Rev ""
+Sheet 9 21
+Title "Mainet-mega -- runReverseControl"
+Date "2021-06-16"
+Rev "1.0"
 Comp ""
 Comment1 ""
@@
 AR Path="/5FC25793/5FF2B76A" Ref="Q?"  Part="1"
 AR Path="/5FC25793/5FF0D186/5FF2B76A" Ref="Q3"  Part="1"
+AR Path="/5FC25793/5FD90F9D/5FF2B76A" Ref="Q3"  Part="1"
 F 0 "Q3" H 6540 4246 50  0000 L CNN
 F 1 "2N3904" H 6540 4155 50  0000 L CNN
@@
 AR Path="/5FC25793/5FF2B770" Ref="R?"  Part="1"
 AR Path="/5FC25793/5FF0D186/5FF2B770" Ref="R6"  Part="1"
+AR Path="/5FC25793/5FD90F9D/5FF2B770" Ref="R6"  Part="1"
 F 0 "R6" V 5793 4200 50  0000 C CNN
 F 1 "R" V 5884 4200 50  0000 C CNN
@@
 AR Path="/5FC25793/5FF2B776" Ref="K?"  Part="1"
 AR Path="/5FC25793/5FF0D186/5FF2B776" Ref="K3"  Part="1"
+AR Path="/5FC25793/5FD90F9D/5FF2B776" Ref="K3"  Part="1"
 F 0 "K3" H 7080 3546 50  0000 L CNN
 F 1 "SANYOU_SRD_Form_C" H 7080 3455 50  0001 L CNN
@@
 AR Path="/5FC25793/5FF2B77C" Ref="D?"  Part="1"
 AR Path="/5FC25793/5FF0D186/5FF2B77C" Ref="D6"  Part="1"
+AR Path="/5FC25793/5FD90F9D/5FF2B77C" Ref="D6"  Part="1"
 F 0 "D6" V 5904 3579 50  0000 L CNN
 F 1 "1N4007" V 5995 3579 50  0000 L CNN
@@
 AR Path="/5FC25793/5FF2B783" Ref="#PWR?"  Part="1"
 AR Path="/5FC25793/5FF0D186/5FF2B783" Ref="#PWR020"  Part="1"
-F 0 "#PWR020" H 6450 2650 50  0001 C CNN
+AR Path="/5FC25793/5FD90F9D/5FF2B783" Ref="#PWR0103"  Part="1"
+F 0 "#PWR0103" H 6450 2650 50  0001 C CNN
 F 1 "+5V" H 6465 2973 50  0000 C CNN
 F 2 "" H 6450 2800 50  0001 C CNN
@@
 AR Path="/5FC25793/5FF2B78A" Ref="U?"  Part="1"
 AR Path="/5FC25793/5FF0D186/5FF2B78A" Ref="U4"  Part="1"
+AR Path="/5FC25793/5FD90F9D/5FF2B78A" Ref="U4"  Part="1"
 F 0 "U4" H 5200 4425 50  0000 C CNN
 F 1 "4N37" H 5200 4334 50  0000 C CNN
@@
 AR Path="/5FC25793/5FF2B794" Ref="D?"  Part="1"
 AR Path="/5FC25793/5FF0D186/5FF2B794" Ref="D5"  Part="1"
+AR Path="/5FC25793/5FD90F9D/5FF2B794" Ref="D5"  Part="1"
 F 0 "D5" H 4493 4416 50  0000 C CNN
 F 1 "LED" H 4493 4325 50  0000 C CNN
@@
 AR Path="/5FC25793/5FF2B79B" Ref="R?"  Part="1"
 AR Path="/5FC25793/5FF0D186/5FF2B79B" Ref="R5"  Part="1"
+AR Path="/5FC25793/5FD90F9D/5FF2B79B" Ref="R5"  Part="1"
 F 0 "R5" V 4693 3650 50  0000 C CNN
 F 1 "R" V 4784 3650 50  0000 C CNN
@@
 AR Path="/5FC25793/5FF2B7AF" Ref="J?"  Part="1"
 AR Path="/5FC25793/5FF0D186/5FF2B7AF" Ref="J36"  Part="1"
-F 0 "J36" H 8168 3567 50  0000 C CNN
+AR Path="/5FC25793/5FD90F9D/5FF2B7AF" Ref="J78"  Part="1"
+F 0 "J78" H 8168 3567 50  0000 C CNN
 F 1 "Screw_Terminal_01x03" H 8168 3566 50  0001 C CNN
 F 2 "" H 8250 3800 50  0001 C CNN
@@
 	7650 3900 8050 3900
 Text Label 7900 3700 0    50   ~ 0
-NO1
+NO3
 Text Label 7900 3800 0    50   ~ 0
-C1
+C3
 Text Label 7900 3900 0    50   ~ 0
-NC1
+NC3
 Wire Wire Line
 	8050 3700 7750 3700
@@
 AR Path="/5FC25793/5FEE9D1F/5FF2B7BF" Ref="#PWR?"  Part="1"
 AR Path="/5FC25793/5FF0D186/5FF2B7BF" Ref="#PWR021"  Part="1"
-F 0 "#PWR021" H 6450 4150 50  0001 C CNN
+AR Path="/5FC25793/5FD90F9D/5FF2B7BF" Ref="#PWR0104"  Part="1"
+F 0 "#PWR0104" H 6450 4150 50  0001 C CNN
 F 1 "GND" H 6455 4227 50  0000 C CNN
 F 2 "" H 6450 4400 50  0001 C CNN
@@
 AR Path="/5FC25793/5FEE9D1F/5FF2B7CB" Ref="#PWR?"  Part="1"
 AR Path="/5FC25793/5FF0D186/5FF2B7CB" Ref="#PWR019"  Part="1"
-F 0 "#PWR019" H 4050 3050 50  0001 C CNN
+AR Path="/5FC25793/5FD90F9D/5FF2B7CB" Ref="#PWR0105"  Part="1"
+F 0 "#PWR0105" H 4050 3050 50  0001 C CNN
 F 1 "GND" H 4055 3127 50  0000 C CNN
 F 2 "" H 4050 3300 50  0001 C CNN
@@
 	1    0    0    -1
 $EndComp
-Text HLabel 3650 3150 0    50   Input ~ 0
-GND
 Wire Wire Line
 	3650 3150 4050 3150
 Wire Wire Line
 	4050 3150 4050 3300
-Text HLabel 3650 3050 0    50   Input ~ 0
-VCC
-Text HLabel 3650 2950 0    50   Input ~ 0
-JD-VCC
-Wire Wire Line
-	3700 3050 4900 3050
 Wire Wire Line
 	4900 3050 4900 3500
@@
 	5600 2950 3650 2950
 Connection ~ 5600 2950
+$Comp
+L Connector:Conn_01x01_Male J?
+U 1 1 60D05CF4
+P 8750 3700
+AR Path="/5FC25793/5FD90A95/60D05CF4" Ref="J?"  Part="1"
+AR Path="/5FC25793/5FD90F9D/60D05CF4" Ref="J86"  Part="1"
+F 0 "J86" H 8750 3850 50  0000 C CNN
+F 1 "Conn_01x01_Male" H 8858 3790 50  0001 C CNN
+F 2 "" H 8750 3700 50  0001 C CNN
+F 3 "~" H 8750 3700 50  0001 C CNN
+	1    8750 3700
+	1    0    0    -1
+$EndComp
+$Comp
+L Connector:Conn_01x01_Male J?
+U 1 1 60D05CFA
+P 8750 3800
+AR Path="/5FC25793/5FD90A95/60D05CFA" Ref="J?"  Part="1"
+AR Path="/5FC25793/5FD90F9D/60D05CFA" Ref="J87"  Part="1"
+F 0 "J87" H 8750 3650 50  0000 C CNN
+F 1 "Conn_01x01_Male" H 8858 3890 50  0001 C CNN
+F 2 "" H 8750 3800 50  0001 C CNN
+F 3 "~" H 8750 3800 50  0001 C CNN
+	1    8750 3800
+	1    0    0    -1
+$EndComp
+$Comp
+L power:+24V #PWR?
+U 1 1 60D05D00
+P 9150 3200
+AR Path="/5FC25793/5FD90A95/60D05D00" Ref="#PWR?"  Part="1"
+AR Path="/5FC25793/5FD90F9D/60D05D00" Ref="#PWR0106"  Part="1"
+F 0 "#PWR0106" H 9150 3050 50  0001 C CNN
+F 1 "+24V" H 9165 3373 50  0000 C CNN
+F 2 "" H 9150 3200 50  0001 C CNN
+F 3 "" H 9150 3200 50  0001 C CNN
+	1    9150 3200
+	1    0    0    -1
+$EndComp
+Wire Wire Line
+	9150 3200 9150 3700
+Wire Wire Line
+	9150 3700 8950 3700
+Text Label 8950 3700 0    50   ~ 0
+NO3
+Text Label 8950 3800 0    50   ~ 0
+C3
+Wire Wire Line
+	8950 3800 9450 3800
+Text GLabel 9450 3800 2    50   Input ~ 0
+Digital_input_4
+Text Notes 10300 3950 2    50   ~ 0
+Terminal 13 del M400
+Text Notes 4350 4450 2    50   ~ 0
+D19-runReverseControl
+Wire Wire Line
+	3650 3050 4900 3050
+Text GLabel 3650 2950 0    50   Input ~ 0
+JD-VCC
+Text GLabel 3650 3150 0    50   Input ~ 0
+GND
+Text GLabel 3650 3050 0    50   Input ~ 0
+VCC
+Text Notes 7750 3050 2    50   ~ 0
+3er relé de izquierda a derecha
 $EndSCHEMATC

Commit message: KICAD: Actualizar archivos del módulo de relés
Other:
- note added: "Relay Ground\nNo conectar a la tierra\ndel Arduino Mega\n"
- note removed: "No conectar a la tierra del Arduino Mega\n"
- note removed: "Relay Ground\n"
Changed lines of the file:
@@
 $Descr A4 11693 8268
 encoding utf-8
-Sheet 9 21
+Sheet 9 22
 Title "Mainet-mega -- runReverseControl"
-Date "2021-06-16"
+Date "2021-06-17"
 Rev "1.0"
 Comp ""
@@
 Text Notes 5900 2550 0    50   ~ 0
 Fuente externa de +5V\n(No es la salida de +5V \ndel Arduino)
-Text Notes 6600 4500 0    50   ~ 0
-Relay Ground\n
-Text Notes 6600 4600 0    50   ~ 0
-No conectar a la tierra del Arduino Mega\n
 NoConn ~ 5500 4000
 Wire Wire Line
@@
 AR Path="/5FC25793/5FD90A95/60D05CF4" Ref="J?"  Part="1"
 AR Path="/5FC25793/5FD90F9D/60D05CF4" Ref="J86"  Part="1"
-F 0 "J86" H 8750 3850 50  0000 C CNN
+F 0 "J86" H 8650 3700 50  0000 C CNN
 F 1 "Conn_01x01_Male" H 8858 3790 50  0001 C CNN
 F 2 "" H 8750 3700 50  0001 C CNN
@@
 AR Path="/5FC25793/5FD90A95/60D05CFA" Ref="J?"  Part="1"
 AR Path="/5FC25793/5FD90F9D/60D05CFA" Ref="J87"  Part="1"
-F 0 "J87" H 8750 3650 50  0000 C CNN
+F 0 "J87" H 8650 3800 50  0000 C CNN
 F 1 "Conn_01x01_Male" H 8858 3890 50  0001 C CNN
 F 2 "" H 8750 3800 50  0001 C CNN
@@
 Text Notes 7750 3050 2    50   ~ 0
 3er relé de izquierda a derecha
+Text Notes 6100 4900 0    50   ~ 0
+Relay Ground\nNo conectar a la tierra\ndel Arduino Mega\n
+Text Notes 3700 3800 0    50   ~ 0
+Relay Ground\nNo conectar a la tierra\ndel Arduino Mega\n
 $EndSCHEMATC

Commit message: KICAD: Agregar cambios esquemáticos
Other:
- note added: "Nota:\nEsta tensión de 24V la proporciona el M400, \nen los terminales 9 y 17."
- note added: "Terminal 9 del M400"
Changed lines of the file:
@@
 Sheet 9 22
 Title "Mainet-mega -- runReverseControl"
-Date "2021-06-17"
+Date "2021-06-18"
 Rev "1.0"
 Comp ""
@@
 $EndComp
 Wire Wire Line
-	9150 3200 9150 3700
+	9150 3200 9150 3300
 Wire Wire Line
 	9150 3700 8950 3700
@@
 Text Notes 3700 3800 0    50   ~ 0
 Relay Ground\nNo conectar a la tierra\ndel Arduino Mega\n
+Text GLabel 9450 3300 2    50   Input ~ 0
+24V_user
+Wire Wire Line
+	9150 3300 9450 3300
+Text Notes 9450 3450 0    50   ~ 0
+Terminal 9 del M400
+Text Notes 9450 3700 0    50   ~ 0
+Nota:\nEsta tensión de 24V la proporciona el M400, \nen los terminales 9 y 17.
+Connection ~ 9150 3300
+Wire Wire Line
+	9150 3300 9150 3700
 $EndSCHEMATC
