File: kicad/mainet-mega-m400.sch (KiCad schematic (older format))
At the start: 5 parts, among them J40 Screw_Terminal_01x04, J64 Screw_Terminal_01x09, J65 Screw_Terminal_01x17, J66 Screw_Terminal_01x02, J88 Screw_Terminal_01x04

Commit message: KICAD: Agregar User_enable_1 al .sch del M400. Así se puede inhibir su funcionamiento desde el SW machineEnable (User_machine_2) y desde el software Ambas señales deben ser HIGH para permitir el funcionamiento del M400
Connections:
- net User_enable_1: now reaches J88.4 (Pin_4)
- no-connect marks 14 -> 13
Changed lines of the file:
@@
 P 3800 4950
 F 0 "J88" V 3764 4662 50  0000 R CNN
-F 1 "Screw_Terminal_01x04" V 3673 4662 50  0000 R CNN
+F 1 "Screw_Terminal_01x04" V 3673 4662 50  0001 R CNN
 F 2 "" H 3800 4950 50  0001 C CNN
 F 3 "~" H 3800 4950 50  0001 C CNN
@@
 Text Notes 4050 2250 2    50   ~ 0
 42
-NoConn ~ 4000 5150
 Text GLabel 5650 4550 0    50   Input ~ 0
 Analog_input_1-
@@
 Wire Wire Line
 	5650 4550 5800 4550
+Text GLabel 4000 5150 3    50   Input ~ 0
+User_enable_1
 $EndSCHEMATC
