File: kicad/frequencyRefControl.sch (KiCad schematic (older format))
At the start: 14 parts, among them J71 Screw_Terminal_01x02, J72 Screw_Terminal_01x04, J83 Conn_01x01_Male, J84 Conn_01x01_Male, J85 Conn_01x01_Male, Q15 BUK9518-55, U14 4N38

Commit message: KICAD: Correguir frequencyRefControl.sch conexión erronea en J72
Connections:
- net GNDD: no longer D24.2 (A), D25.1 (K), J72.1 (Pin_1), J72.3 (Pin_3), U14.5
- new net 10V: D24.2 (A), D25.1 (K), J72.1 (Pin_1), J72.3 (Pin_3), U14.5
Changed lines of the file:
@@
 Sheet 18 22
 Title "Mainet-mega -- frequencyRefControl"
-Date "2021-07-29"
+Date "2021-07-30"
 Rev "1.0"
 Comp "Tovenca"
@@
 Comment4 ""
 $EndDescr
-Wire Wire Line
-	7900 3600 8000 3600
-Connection ~ 7900 3600
 Text Notes 9300 3900 0    50   ~ 0
 Terminal 2 del M400
@@
 Wire Wire Line
 	7900 3700 8000 3700
-Wire Wire Line
-	7600 3600 7900 3600
 Wire Wire Line
 	7900 3500 7900 3600
@@
 Text Notes 1850 4050 0    50   ~ 0
 D13 (frequencyRefControl)
+Wire Wire Line
+	7600 3600 8000 3600
 $EndSCHEMATC

Commit message: KICAD: Cambiar .sch de frequencyRefControl se volvió al diseño original del PWM
Parts:
- added D?: ~, LED_THT:LED_D5.0mm, symbol Device:LED
- added J? (x2): ~, TerminalBlock_Altech:Altech_AK300_1x03_P5.00mm_45-Degree, symbol Connector:Screw_Terminal_01x03
- added Q?: ~, Package_TO_SOT_THT:TO-220-3_Vertical, symbol Transistor_FET:IRLZ44N
- added Q?: ~, Package_TO_SOT_THT:TO-92_Inline, symbol Transistor_BJT:2N3906
- added R?: 1.5K, Resistor_THT:R_Axial_DIN0207_L6.3mm_D2.5mm_P7.62mm_Horizontal, symbol Device:R
- added R?: 1K, Resistor_THT:R_Axial_DIN0207_L6.3mm_D2.5mm_P7.62mm_Horizontal, symbol Device:R
- added R?: 330, Resistor_THT:R_Axial_DIN0207_L6.3mm_D2.5mm_P7.62mm_Horizontal, symbol Device:R
- added R?: 2K, Resistor_THT:R_Axial_DIN0207_L6.3mm_D2.5mm_P7.62mm_Horizontal, symbol Device:R
- added R?: 4.3K, Resistor_THT:R_Axial_DIN0207_L6.3mm_D2.5mm_P7.62mm_Horizontal, symbol Device:R
- added R?: 690, Resistor_THT:R_Axial_DIN0207_L6.3mm_D2.5mm_P7.62mm_Horizontal, symbol Device:R
- added U?: ~, Package_DIP:DIP-6_W7.62mm, symbol Isolator:4N36
Connections:
- net 10V is gone; now on net GNDD: D24.2 (A), D25.1 (K), J72.1 (Pin_1), J72.3 (Pin_3), U14.5
- net 10V_user: now also J?.3 (Pin_3), R?.1, U?.5
- net Analog_input_1+: now also J?.2 (Pin_2), Q?.2 (D), R?.2; no longer D25.2 (A), J72.4 (Pin_4), Q15.2 (D), R38.2
- net GNDD: now also D?.1 (K), J?.1 (Pin_1), J?.3 (Pin_3), Q?.3 (C), Q?.3 (S), R?.1
- new net: D25.2 (A), J72.4 (Pin_4), Q15.2 (D), R38.2
- new net: Q?.1 (G), R?.2, R?.2
- new net: R?.1, U?.1
- new net: Q?.1 (E), U?.2
- new net: R?.1, R?.2, U?.4
- new net: D?.2 (A), R?.1
- new net: Q?.2 (B), R?.1
- new net: J?.2 (Pin_2), R?.2
- new net +5V: J?.1 (Pin_1), R?.2
- no-connect marks 1 -> 2
Other:
- note added: "Blanco/Verde"
- note added: "GNDD"
- note added: "Verde"
- moved on the sheet: D19, D24, D25, J71, J72, Q15, R34, R35, R36, R38, U14

Commit message: KICAD: Agregar valores resistencias
Parts:
- Q18: renamed from Q?; value ~ -> IRF540
- gave numbers to parts that had none: 11
Changed lines of the file:
@@
 AR Path="/5FBD1D9A/61175FE3" Ref="Q?"  Part="1"
 AR Path="/5FBD1D9A/601ACD13/61175FE3" Ref="Q?"  Part="1"
-AR Path="/5FBD1D9A/601C4CB6/61175FE3" Ref="Q?"  Part="1"
-F 0 "Q?" H 7054 3896 50  0000 L CNN
-F 1 "~" H 6850 3850 50  0001 C CNN
+AR Path="/5FBD1D9A/601C4CB6/61175FE3" Ref="Q18"  Part="1"
+F 0 "Q18" H 7054 3896 50  0000 L CNN
+F 1 "IRF540" H 7200 3800 50  0000 C CNN
 F 2 "Package_TO_SOT_THT:TO-220-3_Vertical" H 7100 3775 50  0001 L CIN
 F 3 "http://www.irf.com/product-info/datasheets/data/irlz44n.pdf" H 6850 3850 50  0001 L CNN
@@
 AR Path="/5FBD1D9A/61175FE9" Ref="U?"  Part="1"
 AR Path="/5FBD1D9A/601ACD13/61175FE9" Ref="U?"  Part="1"
-AR Path="/5FBD1D9A/601C4CB6/61175FE9" Ref="U?"  Part="1"
-F 0 "U?" H 5550 4075 50  0000 C CNN
+AR Path="/5FBD1D9A/601C4CB6/61175FE9" Ref="U18"  Part="1"
+F 0 "U18" H 5550 4075 50  0000 C CNN
 F 1 "~" H 5550 3750 50  0001 C CNN
 F 2 "Package_DIP:DIP-6_W7.62mm" H 5350 3550 50  0001 L CIN
@@
 AR Path="/5FBD1D9A/61175FEF" Ref="R?"  Part="1"
 AR Path="/5FBD1D9A/601ACD13/61175FEF" Ref="R?"  Part="1"
-AR Path="/5FBD1D9A/601C4CB6/61175FEF" Ref="R?"  Part="1"
-F 0 "R?" V 6550 4150 50  0000 C CNN
+AR Path="/5FBD1D9A/601C4CB6/61175FEF" Ref="R49"  Part="1"
+F 0 "R49" V 6550 4150 50  0000 C CNN
 F 1 "1.5K" V 6650 4150 50  0000 C CNN
 F 2 "Resistor_THT:R_Axial_DIN0207_L6.3mm_D2.5mm_P7.62mm_Horizontal" V 6580 4150 50  0001 C CNN
@@
 AR Path="/5FBD1D9A/61175FF6" Ref="R?"  Part="1"
 AR Path="/5FBD1D9A/601ACD13/61175FF6" Ref="R?"  Part="1"
-AR Path="/5FBD1D9A/601C4CB6/61175FF6" Ref="R?"  Part="1"
-F 0 "R?" V 6350 3850 50  0000 C CNN
+AR Path="/5FBD1D9A/601C4CB6/61175FF6" Ref="R48"  Part="1"
+F 0 "R48" V 6350 3850 50  0000 C CNN
 F 1 "1K" V 6250 3850 50  0000 C CNN
 F 2 "Resistor_THT:R_Axial_DIN0207_L6.3mm_D2.5mm_P7.62mm_Horizontal" V 6180 3850 50  0001 C CNN
@@
 AR Path="/5FBD1D9A/61175FFF" Ref="D?"  Part="1"
 AR Path="/5FBD1D9A/601ACD13/61175FFF" Ref="D?"  Part="1"
-AR Path="/5FBD1D9A/601C4CB6/61175FFF" Ref="D?"  Part="1"
-F 0 "D?" H 5843 4667 50  0000 C CNN
+AR Path="/5FBD1D9A/601C4CB6/61175FFF" Ref="D21"  Part="1"
+F 0 "D21" H 5843 4667 50  0000 C CNN
 F 1 "~" H 5850 4450 50  0001 C CNN
 F 2 "LED_THT:LED_D5.0mm" H 5850 4450 50  0001 C CNN
@@
 AR Path="/5FBD1D9A/61176005" Ref="R?"  Part="1"
 AR Path="/5FBD1D9A/601ACD13/61176005" Ref="R?"  Part="1"
-AR Path="/5FBD1D9A/601C4CB6/61176005" Ref="R?"  Part="1"
-F 0 "R?" V 5150 3300 50  0000 C CNN
+AR Path="/5FBD1D9A/601C4CB6/61176005" Ref="R46"  Part="1"
+F 0 "R46" V 5150 3300 50  0000 C CNN
 F 1 "330" V 5250 3300 50  0000 C CNN
 F 2 "Resistor_THT:R_Axial_DIN0207_L6.3mm_D2.5mm_P7.62mm_Horizontal" V 5180 3300 50  0001 C CNN
@@
 AR Path="/5FBD1D9A/6117600F" Ref="R?"  Part="1"
 AR Path="/5FBD1D9A/601ACD13/6117600F" Ref="R?"  Part="1"
-AR Path="/5FBD1D9A/601C4CB6/6117600F" Ref="R?"  Part="1"
-F 0 "R?" V 5750 4150 50  0000 C CNN
+AR Path="/5FBD1D9A/601C4CB6/6117600F" Ref="R47"  Part="1"
+F 0 "R47" V 5750 4150 50  0000 C CNN
 F 1 "2K" V 5850 4150 50  0000 C CNN
 F 2 "Resistor_THT:R_Axial_DIN0207_L6.3mm_D2.5mm_P7.62mm_Horizontal" V 5780 4150 50  0001 C CNN
@@
 AR Path="/5FBD1D9A/61176016" Ref="J?"  Part="1"
 AR Path="/5FBD1D9A/601ACD13/61176016" Ref="J?"  Part="1"
-AR Path="/5FBD1D9A/601C4CB6/61176016" Ref="J?"  Part="1"
-F 0 "J?" H 8000 3300 50  0000 C CNN
+AR Path="/5FBD1D9A/601C4CB6/61176016" Ref="J136"  Part="1"
+F 0 "J136" H 8000 3300 50  0000 C CNN
 F 1 "~" H 8000 3600 50  0001 C CNN
 F 2 "TerminalBlock_Altech:Altech_AK300_1x03_P5.00mm_45-Degree" H 8000 3600 50  0001 C CNN
@@
 AR Path="/5FBD1D9A/6117601D" Ref="R?"  Part="1"
 AR Path="/5FBD1D9A/601ACD13/6117601D" Ref="R?"  Part="1"
-AR Path="/5FBD1D9A/601C4CB6/6117601D" Ref="R?"  Part="1"
-F 0 "R?" H 4550 4100 50  0000 C CNN
+AR Path="/5FBD1D9A/601C4CB6/6117601D" Ref="R45"  Part="1"
+F 0 "R45" H 4550 4100 50  0000 C CNN
 F 1 "4.3K" V 4650 4100 50  0000 C CNN
 F 2 "Resistor_THT:R_Axial_DIN0207_L6.3mm_D2.5mm_P7.62mm_Horizontal" V 4580 4100 50  0001 C CNN
@@
 AR Path="/5FBD1D9A/6117602C" Ref="R?"  Part="1"
 AR Path="/5FBD1D9A/601ACD13/6117602C" Ref="R?"  Part="1"
-AR Path="/5FBD1D9A/601C4CB6/6117602C" Ref="R?"  Part="1"
-F 0 "R?" V 7050 3200 50  0000 C CNN
+AR Path="/5FBD1D9A/601C4CB6/6117602C" Ref="R50"  Part="1"
+F 0 "R50" V 7050 3200 50  0000 C CNN
 F 1 "690" V 6950 3200 50  0000 C CNN
 F 2 "Resistor_THT:R_Axial_DIN0207_L6.3mm_D2.5mm_P7.62mm_Horizontal" V 6880 3200 50  0001 C CNN
@@
 P 5150 4250
 AR Path="/5FBD1D9A/601ACD13/61176038" Ref="Q?"  Part="1"
-AR Path="/5FBD1D9A/601C4CB6/61176038" Ref="Q?"  Part="1"
-F 0 "Q?" H 5340 4204 50  0000 L CNN
+AR Path="/5FBD1D9A/601C4CB6/61176038" Ref="Q14"  Part="1"
+F 0 "Q14" H 5340 4204 50  0000 L CNN
 F 1 "~" H 5150 4250 50  0001 C CNN
 F 2 "Package_TO_SOT_THT:TO-92_Inline" H 5350 4175 50  0001 L CIN
@@
 AR Path="/5FBD1D9A/61176040" Ref="J?"  Part="1"
 AR Path="/5FBD1D9A/601ACD13/61176040" Ref="J?"  Part="1"
-AR Path="/5FBD1D9A/601C4CB6/61176040" Ref="J?"  Part="1"
-F 0 "J?" H 3600 4150 50  0000 C CNN
+AR Path="/5FBD1D9A/601C4CB6/61176040" Ref="J135"  Part="1"
+F 0 "J135" H 3600 4150 50  0000 C CNN
 F 1 "~" H 3600 3850 50  0001 C CNN
 F 2 "TerminalBlock_Altech:Altech_AK300_1x03_P5.00mm_45-Degree" H 3600 3850 50  0001 C CNN
