File: kicad/mainet-mega-control-relay.sch (KiCad schematic (older format))
At the start: 0 parts

Commit message: KICAD: Corregir numeración pines Arduino de control de relés
Other:
- note added: "D0"
- note added: "D1"
- note added: "D2"
- note added: "D3"
- note added: "D4"
- note added: "D5"
- note added: "D6"
- note removed: "D15"
- note removed: "D16"
- note removed: "D17"
- note removed: "D18"
- note removed: "D19"
- note removed: "D20"
- note removed: "D21"
Changed lines of the file:
@@
 brakeChuckControl
 Text Notes 4050 850  0    50   ~ 0
-D21
+D0
 Text Notes 4200 1700 0    50   ~ 0
-D20
+D1
 Text Notes 4200 2600 0    50   ~ 0
-D19
+D2
 Text Notes 3950 3500 0    50   ~ 0
-D18
+D3
 Text Notes 4200 4450 0    50   ~ 0
-D17
+D4
 Text Notes 4150 5400 0    50   ~ 0
-D16
+D5
 Text Notes 4200 6350 0    50   ~ 0
-D15
+D6
 $EndSCHEMATC
