File: kicad/mainet-mega-5V-to-mp-10v.kicad_pcb (KiCad board)
At the start: 2 copper layers, 43.2 x 67.3 mm, 12 parts, among them J1 Screw_Terminal_01x03, J2 Screw_Terminal_01x03, Q1 2N3906, Q2 BUK9518-55, U1 4N38

Commit message: Modificar pcb
Routing:
- net Net-(Q1-Pad1): track 20.6 -> 21.8 mm

Commit message: Corregir numeración de pines terminales J2 / PCB
Connections:
- J2 pad 1: /0V -> /+10V
- J2 pad 3: /+10V -> /0V
Changed lines of the file:
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@@
   (layers
     (0 F.Cu signal hide)
-    (31 B.Cu signal hide)
+    (31 B.Cu signal)
     (32 B.Adhes user hide)
     (33 F.Adhes user hide)
@@
     (mod_text_size 1 1)
     (mod_text_width 0.15)
-    (pad_size 2 3)
-    (pad_drill 0.9)
+    (pad_size 4 5)
+    (pad_drill 1.5)
     (pad_to_mask_clearance 0)
     (aux_axis_origin 0 0)
@@
       (effects (font (size 1 1) (thickness 0.15)))
     )
-    (pad 1 thru_hole oval (at 0 0) (size 4 5) (drill 1.5) (layers *.Cu *.Mask)
+    (pad 3 thru_hole oval (at 0 0) (size 4 5) (drill 1.5) (layers *.Cu *.Mask)
       (net 1 /0V))
     (pad 2 thru_hole oval (at 5 0) (size 4 5) (drill 1.5) (layers *.Cu *.Mask)
       (net 6 "Net-(J2-Pad2)"))
-    (pad 3 thru_hole rect (at 10 0) (size 4 5) (drill 1.5) (layers *.Cu *.Mask)
+    (pad 1 thru_hole rect (at 10 0) (size 4 5) (drill 1.5) (layers *.Cu *.Mask)
       (net 7 /+10V))
     (model ${KISYS3DMOD}/TerminalBlock_Altech.3dshapes/Altech_AK300_1x03_P5.00mm_45-Degree.wrl
